File: pcb/plaid.kicad_pcb (KiCad board)
At the start: 2 copper layers, 228 x 98 mm, 138 parts, among them J1 USB_OTG, J2 AVR_ISP_6, J3 Conn_01x04, J4 GS2, J5 GS2, SW1 SW_Push, SW10 SW_Push, SW11 SW_Push, SW12 SW_Push, SW13 SW_Push, SW14 SW_Push, SW15 SW_Push, SW16 SW_Push, SW17 SW_Push, SW18 SW_Push, SW19 SW_Push, SW2 SW_Push, SW20 SW_Push, SW21 SW_Push, SW22 SW_Push, SW23 SW_Push, SW24 SW_Push, SW25 SW_Push, SW26 SW_Push, SW27 SW_Push, SW28 SW_Push, SW29 SW_Push, SW3 SW_Push, SW30 SW_Push, SW31 SW_Push, SW32 SW_Push, SW33 SW_Push, SW34 SW_Push, SW35 SW_Push, SW36 SW_Push, SW37 SW_Push, SW38 SW_Push, SW39 SW_Push, SW4 SW_Push, SW40 SW_Push, SW41 SW_Push, SW42 SW_Push, SW43 SW_Push, SW44 SW_Push, SW45 SW_Push, SW46 SW_Push, SW47 SW_Push, SW48 SW_Push, SW49 SW_Push, SW5 SW_Push, SW50 RESET, SW51 BOOT, SW6 SW_Push, SW7 SW_Push, SW8 SW_Push, SW9 SW_Push, U1 ATMEGA328-PU, Y1 16MHz

Commit message: update pcb add readme.md
Routing:
- net Net-(D32-Pad2): track 86.7 -> 87.7 mm
- net Net-(D43-Pad2): track 108.0 -> 108.8 mm
- net Net-(D20-Pad2): track 71.9 -> 72.7 mm
- net Net-(D45-Pad2): track 129.4 -> 128.7 mm
