File: pcb/plaid.kicad_pcb (KiCad board)
At the start: 2 copper layers, 228 x 98 mm, 138 parts, among them J1 USB_OTG, J2 AVR_ISP_6, J3 Conn_01x04, J4 GS2, J5 GS2, SW1 SW_Push, SW10 SW_Push, SW11 SW_Push, SW12 SW_Push, SW13 SW_Push, SW14 SW_Push, SW15 SW_Push, SW16 SW_Push, SW17 SW_Push, SW18 SW_Push, SW19 SW_Push, SW2 SW_Push, SW20 SW_Push, SW21 SW_Push, SW22 SW_Push, SW23 SW_Push, SW24 SW_Push, SW25 SW_Push, SW26 SW_Push, SW27 SW_Push, SW28 SW_Push, SW29 SW_Push, SW3 SW_Push, SW30 SW_Push, SW31 SW_Push, SW32 SW_Push, SW33 SW_Push, SW34 SW_Push, SW35 SW_Push, SW36 SW_Push, SW37 SW_Push, SW38 SW_Push, SW39 SW_Push, SW4 SW_Push, SW40 SW_Push, SW41 SW_Push, SW42 SW_Push, SW43 SW_Push, SW44 SW_Push, SW45 SW_Push, SW46 SW_Push, SW47 SW_Push, SW48 SW_Push, SW49 SW_Push, SW5 SW_Push, SW50 RESET, SW51 BOOT, SW6 SW_Push, SW7 SW_Push, SW8 SW_Push, SW9 SW_Push, U1 ATMEGA328-PU, Y1 16MHz

Commit message: Plaid Rev.1 Release
Parts:
- added REF**: Stab_MX_2u, SMKJP:Stab_MX_2u, F.Cu at (164.0, 138.5)
- C3: value 4.7u -> 10u
- C4, C5: footprint Capacitors_THT:C_Disc_D3.0mm_W1.6mm_P2.50mm -> Capacitors_THT:C_Disc_D4.3mm_W1.9mm_P5.00mm
- F1: value 250mA -> 100mA
- R2, R3: value 68R -> 75R
- SW49: footprint SMKJP:SW_Cherry_MX1A_1.00u_PCB -> SMKJP:SW_Cherry_MX1A_2.0U_PCB_universal_center
- moved R4 8.70 mm to (195.5, 61.5), turned to 0 degrees
- moved J2 0.51 mm to (195.5, 69.0)
- renumbered D48 to D42, D42 to D43, D43 to D44, D44 to D45, D45 to D46, D46 to D47, D47 to D48
Routing:
- net /COL7: track 98.8 -> 100.6 mm, vias 1 -> 0
- net /COL8: track 80.1 -> 81.6 mm
- net +5V: track 128.9 -> 127.6 mm
- net /COL6: track 125.8 -> 127.0 mm
- net /RESET: track 72.2 -> 71.3 mm, vias 1 -> 0
- net Net-(D30-Pad2): track 82.1 -> 81.4 mm
- net Net-(D42-Pad2): track 111.5 -> 110.8 mm
- net GND: vias 77 -> 79
Other:
- board text added: "Plaid // Through Hole // Rev.1 (c)2019 Takuya Urakawa, Dm9Records.com"
- board text removed: "Plaid // Through Hole // Rev.Alpha (c)2018 Takuya Urakawa, Dm9Records.com"

Commit message: Add files via upload
Parts:
- moved SW51 7.97 mm to (194.6, 53.8), turned to 0 degrees
- moved R4 5.07 mm to (200.6, 61.9), turned to 180 degrees
- moved G*** 0.23 mm to (119.7, 51.2)
Routing:
- net GND: track 8.83 -> 87.5 mm, vias 79 -> 0
- net /COL3: track 180.9 -> 252.4 mm
- net /COL0: track 224.7 -> 273.9 mm, vias 1 -> 0
- net /COL1: track 217.0 -> 257.9 mm
- net /ROW1: track 162.9 -> 202.2 mm
- net /ROW0: track 156.3 -> 194.5 mm
- net /COL8: track 81.6 -> 115.5 mm
- net /COL4: track 168.5 -> 199.4 mm
- net /COL6: track 127.0 -> 157.7 mm, vias 1 -> 0
- net /COL7: track 100.6 -> 130.7 mm
- net Net-(D8-Pad2): track 75.4 -> 105.4 mm, vias 1 -> 0
- net /RESET: track 71.3 -> 101.0 mm
- net /COL2: track 214.2 -> 243.1 mm
- net /COL5: track 158.5 -> 182.0 mm
- net /ROW2: track 157.5 -> 176.9 mm
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