File: pcb/plaid.kicad_pcb (KiCad board)
At the start: 2 copper layers, 228 x 98 mm, 139 parts, among them J1 USB_OTG, J2 AVR_ISP_6, J3 Conn_01x04, J4 GS2, J5 GS2, SW1 SW_Push, SW10 SW_Push, SW11 SW_Push, SW12 SW_Push, SW13 SW_Push, SW14 SW_Push, SW15 SW_Push, SW16 SW_Push, SW17 SW_Push, SW18 SW_Push, SW19 SW_Push, SW2 SW_Push, SW20 SW_Push, SW21 SW_Push, SW22 SW_Push, SW23 SW_Push, SW24 SW_Push, SW25 SW_Push, SW26 SW_Push, SW27 SW_Push, SW28 SW_Push, SW29 SW_Push, SW3 SW_Push, SW30 SW_Push, SW31 SW_Push, SW32 SW_Push, SW33 SW_Push, SW34 SW_Push, SW35 SW_Push, SW36 SW_Push, SW37 SW_Push, SW38 SW_Push, SW39 SW_Push, SW4 SW_Push, SW40 SW_Push, SW41 SW_Push, SW42 SW_Push, SW43 SW_Push, SW44 SW_Push, SW45 SW_Push, SW46 SW_Push, SW47 SW_Push, SW48 SW_Push, SW49 SW_Push, SW5 SW_Push, SW50 RESET, SW51 BOOT, SW6 SW_Push, SW7 SW_Push, SW8 SW_Push, SW9 SW_Push, U1 ATMEGA328-PU, Y1 16MHz

Commit message: Add files via upload
Parts:
- moved R4 0.46 mm to (200.6, 61.4)
- moved G*** 0.23 mm to (119.7, 51.0)
- moved SW51 0.10 mm to (194.7, 53.8)
Routing:
- net Net-(D43-Pad2): track 110.5 -> 131.3 mm
- net /ROW0: track 194.5 -> 207.2 mm
- net /ROW2: track 176.9 -> 186.6 mm
- net /ROW3: track 181.8 -> 191.0 mm
- net GND: track 87.5 -> 94.3 mm
- net Net-(D10-Pad2): track 97.3 -> 91.2 mm
- net /COL0: track 273.9 -> 278.4 mm
- net Net-(D8-Pad2): track 105.4 -> 101.4 mm
- net Net-(D46-Pad2): track 133.2 -> 129.8 mm
- net +5V: track 132.0 -> 135.2 mm
- net Net-(D40-Pad2): track 90.2 -> 87.1 mm
- net Net-(D31-Pad2): track 88.7 -> 85.7 mm
- net Net-(D19-Pad2): track 66.5 -> 63.6 mm
- net Net-(D16-Pad2): track 44.1 -> 41.7 mm
- net Net-(D4-Pad2): track 23.8 -> 21.6 mm
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